File: circuit/circuit.brd (EAGLE design)
At the start: 100 x 80 mm, 76 parts

Commit message: updated circuit   + layout is done   + updated export files
Parts:
- added JT: (no value), pinhead:1X04
- RD2: value 10k -> 100k
- moved LD1 64.8 mm to (85.1, 5.71), turned to 90 degrees
- moved LD2 64.8 mm to (80.0, 5.71), turned to 270 degrees
- moved RLD1 64.8 mm to (85.1, 14.6)
- moved RLD2 64.8 mm to (80.0, 14.6), turned to 270 degrees
- moved RD8 16.6 mm to (82.5, 14.6), turned to 270 degrees
- moved DD1 6.35 mm to (68.6, 9.53)
- moved RD1 6.35 mm to (59.7, 13.3)
- moved RD5 6.35 mm to (69.8, 5.08)
- moved CD2 6.35 mm to (48.3, 18.4)
- moved DD2 6.35 mm to (62.2, 13.3)
- moved JD1 6.35 mm to (61.0, 5.08)
- moved JD2 6.35 mm to (43.2, 5.08)
- moved JD3 6.35 mm to (25.4, 5.08)
- moved RD2 6.35 mm to (57.1, 13.3)
- moved RD3 6.35 mm to (52.1, 13.3)
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- renumbered JP5 to JP6
Connections:
- net +5V: now also LD1.A
- net BUS_ENABLE: now also RLD2.1; no longer LD2.A
- net BUS_RX: now also RLD1.2; no longer LD1.K
- net GND: now also LD2.K; no longer RLD1.2, RLD2.2
- net N$34: now also LD1.K, RLD1.1; no longer LD2.K, RLD2.1
- net N$37: now also LD2.A, RLD2.2; no longer LD1.A, RLD1.1
- net TWI_SCL: now also JT.1, JT.4
- net TWI_SDA: now also JT.2, JT.3
Routing:
- net +5V: track 524.5 -> 608.5 mm, vias 8 -> 7
- net BTN1: track 6.35 -> 74.8 mm
- net LED1_R: track 2.54 -> 46.1 mm
- net IRLED2_MOSI: track 42.4 -> 85.0 mm, vias 0 -> 1
- net IRLED1: track 0.00 -> 39.0 mm, vias 0 -> 1
- net GND: track 626.1 -> 662.9 mm, vias 9 -> 11
- net LED1_G: track 2.54 -> 39.0 mm
- net LED1_B: track 2.54 -> 33.1 mm
- net TWI_SCL: track 0.00 -> 15.1 mm
- net BUS_RX: track 38.5 -> 51.7 mm
- net TWI_SDA: track 0.00 -> 11.8 mm
- net ICS_TAB: track 0.00 -> 11.8 mm, vias 0 -> 17
- net N$2: track 10.2 -> 3.81 mm
- net BUS_DETECT2: track 14.2 -> 18.8 mm
- net N$46: track 0.00 -> 3.81 mm
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- added copper zone on layer 1, net GND
- added copper zone on layer 16, net GND
- added copper zone on layer 1, net ICS_TAB
- added copper zone on layer 16, net ICS_TAB
Other:
- board text added: "09.01.17"
- board text added: "12V"
- board text added: "5V"
- board text added: "B1"
- board text added: "B2"
- board text added: "BM"
- board text added: "IR1"
- board text added: "IR2"
- board text added: "P. Weissig"
- board text added: "PullDown"
- board text added: "PullUp"
- board text added: "PvP"
- board text added: "R X"
- board text added: "RGB1"
- board text added: "RGB2"
- board text added: "RoboSAX"
- board text added: "T X"
- board text added: "TWI"
- board text added: "Term"

Commit message: finished layout and exported data
Parts:
- added JD4: (no value), pinhead:1X02
- moved CB1 48.6 mm to (26.0, 61.0), turned to 0 degrees
Connections:
- net BUS_DETECT1: now also JD4.2
- net LED2_R: now also JD4.1
Routing:
- net BUS_DETECT1: track 20.5 -> 41.1 mm
- net GND: track 662.9 -> 675.6 mm
- net BTN1: track 74.8 -> 79.7 mm
- net ICS_TAB: track 11.8 -> 8.19 mm, vias 17 -> 21
- net LED2_R: track 71.2 -> 74.4 mm
- net IRLED2_MOSI: track 85.0 -> 85.8 mm
Other:
- board text added: "10.01.17"
- board text removed: "09.01.17"
