File: circuit/full/circuit.brd (EAGLE design)
At the start: 100 x 80 mm, 78 parts

Commit message: switched color of LD1 and LD2 in full version
Parts:
- LD1: value green -> red
- LD2: value red -> green
Changed lines of the file:
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@@
 </element>
 <element name="J202" library="robo_ag" package="STECKER_WANNE_10" value="" x="94.615" y="20.32" rot="R90"/>
-<element name="LD2" library="robo_ag" package="LED_3MM" value="red" x="80.01" y="5.715" smashed="yes" rot="R270">
+<element name="LD2" library="robo_ag" package="LED_3MM" value="green" x="80.01" y="5.715" smashed="yes" rot="R270">
 <attribute name="NAME" x="78.4225" y="1.9685" size="1.27" layer="25" ratio="10"/>
 <attribute name="VALUE" x="78.359" y="3.81" size="1.27" layer="27" ratio="10" rot="R270"/>
@@
 <attribute name="VALUE" x="79.375" y="16.8656" size="1.27" layer="27" ratio="10" rot="R270"/>
 </element>
-<element name="LD1" library="robo_ag" package="LED_3MM" value="green" x="85.09" y="5.715" smashed="yes" rot="R90">
+<element name="LD1" library="robo_ag" package="LED_3MM" value="red" x="85.09" y="5.715" smashed="yes" rot="R90">
 <attribute name="NAME" x="83.82" y="1.9685" size="1.27" layer="25" ratio="10"/>
 <attribute name="VALUE" x="86.741" y="7.62" size="1.27" layer="27" ratio="10" rot="R90"/>
